File: panel.kicad_pcb (KiCad board)
At the start: 2 copper layers, 104.6 x 74.4 mm, 114 parts, among them J1 JST_SH_SM06B-SRSS-TB_1x06-1MP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, J4 Conn_01x04, Q1 BSS84, U1 M24C02-FMN

Commit message: Fix the design around MOSFET and add resistor in series to protect MCU's GPIO line
Parts:
- removed the Q1 at (71.9, 37.8)
- removed the Q1 at (71.9, 68.0)
- removed the Q1 at (132.3, 37.8)
- removed the Q1 at (132.3, 68.0)
- removed the Q1 at (102.1, 37.8)
- removed the Q1 at (102.1, 68.0)
- removed R21 (x6): 10K, Resistor_SMD:R_0603_1608Metric
- removed R23 (x6): 330, Resistor_SMD:R_0603_1608Metric
- added Q1: BSS84, Package_TO_SOT_SMD:SOT-23, F.Cu at (71.7, 67.1)
- added Q1: BSS84, Package_TO_SOT_SMD:SOT-23, F.Cu at (101.9, 36.9)
- added Q1: BSS84, Package_TO_SOT_SMD:SOT-23, F.Cu at (101.9, 67.1)
- added Q1: BSS84, Package_TO_SOT_SMD:SOT-23, F.Cu at (132.1, 67.1)
- added Q1: BSS84, Package_TO_SOT_SMD:SOT-23, F.Cu at (71.7, 36.9)
- added Q1: BSS84, Package_TO_SOT_SMD:SOT-23, F.Cu at (132.1, 36.9)
- added R1: 330, Resistor_SMD:R_0603_1608Metric, F.Cu at (76.3, 67.1)
- added R1: 330, Resistor_SMD:R_0603_1608Metric, F.Cu at (76.3, 36.9)
- added R1: 330, Resistor_SMD:R_0603_1608Metric, F.Cu at (106.5, 67.1)
- added R1: 330, Resistor_SMD:R_0603_1608Metric, F.Cu at (106.5, 36.9)
- added R1: 330, Resistor_SMD:R_0603_1608Metric, F.Cu at (136.8, 36.9)
- added R1: 330, Resistor_SMD:R_0603_1608Metric, F.Cu at (136.8, 67.1)
- added R2: 330, Resistor_SMD:R_0603_1608Metric, F.Cu at (130.3, 42.1)
- added R2: 330, Resistor_SMD:R_0603_1608Metric, F.Cu at (100.1, 72.3)
- added R2: 330, Resistor_SMD:R_0603_1608Metric, F.Cu at (69.9, 42.1)
- added R2: 330, Resistor_SMD:R_0603_1608Metric, F.Cu at (69.9, 72.3)
- added R2: 330, Resistor_SMD:R_0603_1608Metric, F.Cu at (100.1, 42.1)
- added R2: 330, Resistor_SMD:R_0603_1608Metric, F.Cu at (130.3, 72.3)
- added R3: 10K, Resistor_SMD:R_0603_1608Metric, F.Cu at (104.9, 67.1)
- added R3: 10K, Resistor_SMD:R_0603_1608Metric, F.Cu at (74.7, 67.1)
- added R3: 10K, Resistor_SMD:R_0603_1608Metric, F.Cu at (74.7, 36.9)
- added R3: 10K, Resistor_SMD:R_0603_1608Metric, F.Cu at (135.1, 67.1)
- added R3: 10K, Resistor_SMD:R_0603_1608Metric, F.Cu at (104.9, 36.9)
- added R3: 10K, Resistor_SMD:R_0603_1608Metric, F.Cu at (135.1, 36.9)
- R5 (x6), R6 (x6): value 2.2K -> 4.7K
Routing:
- net Board_4-Net-(Q1-D): track 0.00 -> 4.72 mm
- net Board_1-Net-(Q1-D): track 0.00 -> 4.72 mm
- net Board_5-Net-(Q1-D): track 0.00 -> 4.72 mm
- net Board_3-Net-(Q1-D): track 0.00 -> 4.72 mm
- net Board_2-Net-(Q1-D): track 0.00 -> 4.72 mm
- net Board_0-Net-(Q1-D): track 0.00 -> 4.72 mm
- net Board_2-Net-(Q1-S): track 4.55 -> 0.00 mm
- net Board_1-Net-(Q1-S): track 4.55 -> 0.00 mm
- net Board_0-Net-(Q1-S): track 4.55 -> 0.00 mm
- net Board_5-Net-(Q1-S): track 4.55 -> 0.00 mm
- net Board_4-Net-(Q1-S): track 4.55 -> 0.00 mm
- net Board_3-Net-(Q1-S): track 4.55 -> 0.00 mm
- net Board_4-Net-(Q1-G): track 0.00 -> 3.81 mm
- net Board_3-Net-(Q1-G): track 0.00 -> 3.81 mm
- net Board_5-Net-(Q1-G): track 0.00 -> 3.81 mm
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